Commit message: [FDL] finish

File: model/phasespace.urdf.xacro (robot description, xacro)
@@ -46,5 +46,5 @@
 			<child link="${name}_erste_link_x"/>
 			<axis xyz="1 0 0"/>
-			<limit lower="${0}" upper="${1}" effort="${effort}" velocity="${velocity}"/>
+			<limit lower="${0}" upper="${2}" effort="${effort}" velocity="${velocity}"/>
 		</joint>
 		<!-- fake link -->
@@ -57,5 +57,5 @@
 			<child link="${name}_erste_link_y"/>
 			<axis xyz="0 1 0"/>
-			<limit lower="${0}" upper="${1}" effort="${effort}" velocity="${velocity}"/>
+			<limit lower="${0}" upper="${2}" effort="${effort}" velocity="${velocity}"/>
 		</joint>
 		<!-- fake link -->
@@ -68,5 +68,5 @@
 			<child link="${name}_erste_link_z"/>
 			<axis xyz="0 0 1"/>
-			<limit lower="${0}" upper="${1}" effort="${effort}" velocity="${velocity}"/>
+			<limit lower="${0}" upper="${2}" effort="${effort}" velocity="${velocity}"/>
 		</joint>
 		<!-- fake link -->
